File: beaglelogic-standalone.sch (KiCad schematic (older format))
At the start: 247 parts, among them J1 USB_OTG, J2 CONN_02X02, J3 USB_A, J4 CONN_01X06, J5 SI-51009-F, J6 CONN_02X12, J7 CONN_02X16, Q1 BSS138, Q2 BSS138, SW1 SW_PUSH_SMALL_H, SW2 SW_PUSH_SMALL_H, U1 74LVC1G07, U10 MCP79410/TDFN, U11 SST26VF064B, U12 TPS73101, U13 SN74LVCH16T245, U14 DVIULC6-4SC6, U15 DVIULC6-4SC6, U16 DVIULC6-4SC6, U17 DVIULC6-4SC6, U18 74LV1T125, U19 EMMC_4G, U2 AP1117, U3 TPS2051C, U4 TPD4S012, U5 TPD4S012, U6 OSD3358-SM, U7 KSZ9031RNXCC, U8 74LVC2G241, U9 74LVC1G125, Y1 25MHz, Y2 24MHz, Y3 32.768kHz,CL=9pF

Commit message: Footprint assignment completed
All footprints assigned.

Signed-off-by: Kumar Abhishek <abhishek@theembeddedkitchen.net>
Parts:
- J2: footprint (none) -> Pin_Headers:Pin_Header_Straight_2x02_Pitch2.54mm
- J5: footprint (none) -> beaglelogic-standalone:SI-51009-F
- U4, U5: footprint (none) -> beaglelogic-standalone:DRY

Commit message: Schematic changes... 	* Flip D0 to D15 and PRU_IN0 to PRU_IN15 for ease in board layout 	* Switch OSD3358-SM from 400pin BGA to 256pin BGA package
Signed-off-by: Kumar Abhishek <abhishek@theembeddedkitchen.net>
Parts:
- U6: footprint beaglelogic-standalone:BGA-400-1-27mm -> beaglelogic-standalone:BGA-256-1-27mm
Connections:
- net DIN00: now also U13.23 (2B8); no longer U13.2 (1B1)
- net DIN01: now also U13.22 (2B7); no longer U13.3 (1B2)
- net DIN02: now also U13.20 (2B6); no longer U13.5 (1B3)
- net DIN03: now also U13.19 (2B5); no longer U13.6 (1B4)
- net DIN04: now also U13.17 (2B4); no longer U13.8 (1B5)
- net DIN05: now also U13.16 (2B3); no longer U13.9 (1B6)
- net DIN06: now also U13.14 (2B2); no longer U13.11 (1B7)
- net DIN07: now also U13.13 (2B1); no longer U13.12 (1B8)
- net DIN08: now also U13.12 (1B8); no longer U13.13 (2B1)
- net DIN09: now also U13.11 (1B7); no longer U13.14 (2B2)
- net DIN10: now also U13.9 (1B6); no longer U13.16 (2B3)
- net DIN11: now also U13.8 (1B5); no longer U13.17 (2B4)
- net DIN12: now also U13.6 (1B4); no longer U13.19 (2B5)
- net DIN13: now also U13.5 (1B3); no longer U13.20 (2B6)
- net DIN14: now also U13.3 (1B2); no longer U13.22 (2B7)
- net DIN15: now also U13.2 (1B1); no longer U13.23 (2B8)
- net D_RX: no longer J4.5 (P5), U8.3 (2Y)
- net PRU1_IN00: now also U13.26 (2A8); no longer U13.47 (1A1)
- net PRU1_IN01: now also U13.27 (2A7); no longer U13.46 (1A2)
- net PRU1_IN02: now also U13.29 (2A6); no longer U13.44 (1A3)
- net PRU1_IN03: now also U13.30 (2A5); no longer U13.43 (1A4)
- net PRU1_IN04: now also U13.32 (2A4); no longer U13.41 (1A5)
- net PRU1_IN05: now also U13.33 (2A3); no longer U13.40 (1A6)
- net PRU1_IN06: now also U13.35 (2A2); no longer U13.38 (1A7)
- net PRU1_IN07: now also U13.36 (2A1); no longer U13.37 (1A8)
- net PRU1_IN08: now also U13.37 (1A8); no longer U13.36 (2A1)
- net PRU1_IN09: now also U13.38 (1A7); no longer U13.35 (2A2)
- net PRU1_IN10: now also U13.40 (1A6); no longer U13.33 (2A3)
- net PRU1_IN11: now also U13.41 (1A5); no longer U13.32 (2A4)
- net PRU1_IN12: now also U13.43 (1A4); no longer U13.30 (2A5)
- net PRU1_IN13: now also U13.44 (1A3); no longer U13.29 (2A6)
- net PRU1_IN14: now also U13.46 (1A2); no longer U13.27 (2A7)
- net PRU1_IN15: now also U13.47 (1A1); no longer U13.26 (2A8)
- new net D_TX: J4.5 (P5), U8.3 (2Y)
