File: beaglelogic-standalone.kicad_pcb (KiCad board)
At the start: 4 copper layers, 100 x 74 mm, 260 parts, among them J1 USB_OTG, J2 CONN_02X02, J3 USB_A, J4 CONN_01X06, J5 SI-51009-F, J6 CONN_02X12, J7 CONN_02X16, J8 Barrel_Jack, M1 TEST_1P, M2 TEST_1P, M3 TEST_1P, M4 TEST_1P, Q1 BSS138, Q2 BSS138, SW1 SW_PUSH_SMALL_H, SW2 SW_PUSH_SMALL_H, U1 74LVC1G07, U10 MCP79410/TDFN, U11 SST26VF064B, U12 TPS73101, U13 SN74LVCH16T245, U14 DVIULC6-4SC6, U15 DVIULC6-4SC6, U16 DVIULC6-4SC6, U17 DVIULC6-4SC6, U18 74LV1T125, U19 EMMC_4G, U2 AP1117, U3 TPS2051C, U4 TPD4S012, U5 TPD4S012, U6 OSD3358-SM, U7 KSZ9031RNXCC, U8 74LVC2G241, U9 74LVC1G125, Y1 25MHz, Y2 24MHz, Y3 32.768kHz,CL=9pF

Commit message: Release PCB rev A1
Signed-off-by: Kumar Abhishek <abhishek@theembeddedkitchen.net>
Routing:
- net GND: track 556.6 -> 541.2 mm
Other:
- board text added: "Breakaway rails for SMT Production: Do NOT remove until assembly"
Changed lines of the file:
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@@
   (general
     (thickness 1.6)
-    (drawings 141)
-    (tracks 3992)
+    (drawings 145)
+    (tracks 3982)
     (zones 0)
     (modules 260)
@@
     (tags "capacitor 0402")
     (attr smd)
-    (fp_text reference C20 (at 2.2 0 180) (layer F.SilkS)
+    (fp_text reference C20 (at 2 -0.1 180) (layer F.SilkS)
       (effects (font (size 0.7 0.7) (thickness 0.15)))
     )
@@
       (net 1 GND))
   )
+  (gr_text "Breakaway rails for SMT Production: Do NOT remove until assembly" (at 150.9 135.1) (layer B.SilkS)
+    (effects (font (size 1.6 1.6) (thickness 0.3)) (justify mirror))
+  )
+  (gr_text "Breakaway rails for SMT Production: Do NOT remove until assembly" (at 151 66.7) (layer B.SilkS)
+    (effects (font (size 1.6 1.6) (thickness 0.3)) (justify mirror))
+  )
+  (gr_text "Breakaway rails for SMT Production: Do NOT remove until assembly" (at 150.9 135) (layer F.SilkS)
+    (effects (font (size 1.6 1.6) (thickness 0.3)))
+  )
+  (gr_text "Breakaway rails for SMT Production: Do NOT remove until assembly" (at 151 66.8) (layer F.SilkS)
+    (effects (font (size 1.6 1.6) (thickness 0.3)))
+  )
   (gr_arc (start 197.5 131.5) (end 197.5 131) (angle -180) (layer Edge.Cuts) (width 0.2))
   (gr_line (start 197.5 132) (end 201 132) (layer Edge.Cuts) (width 0.2))
@@
   (via (at 108.25 71) (size 1) (drill 0.8) (layers F.Cu B.Cu) (net 0))
   (segment (start 195.4 64) (end 195.4 64.2) (width 0.1524) (layer B.Cu) (net 0))
+  (segment (start 124.6 107.95) (end 124.6 108.4024) (width 0.1524) (layer B.Cu) (net 1))
+  (segment (start 124.6 108.4024) (end 124.8976 108.7) (width 0.1524) (layer B.Cu) (net 1))
+  (segment (start 124.8976 108.7) (end 131.9 108.7) (width 0.1524) (layer B.Cu) (net 1))
+  (segment (start 131.9 108.7) (end 132.1 108.5) (width 0.1524) (layer B.Cu) (net 1))
+  (segment (start 132.1 108.5) (end 132.1 107.95) (width 0.1524) (layer B.Cu) (net 1))
   (segment (start 127.5 93.65) (end 124.35935 93.65) (width 0.381) (layer F.Cu) (net 1))
   (segment (start 124.35935 93.65) (end 122.906175 95.103175) (width 0.381) (layer F.Cu) (net 1))
@@
   (segment (start 155.1524 114.35) (end 155.4 114.1024) (width 0.1524) (layer F.Cu) (net 1))
   (segment (start 155.4 113.5) (end 155.2 113.5) (width 0.1524) (layer F.Cu) (net 1))
-  (segment (start 155.2 113.5) (end 155.025 113.5) (width 0.1524) (layer F.Cu) (net 1))
-  (segment (start 154.85 112.6) (end 154.65 112.4) (width 0.1524) (layer F.Cu) (net 1))
-  (segment (start 154.85 113.325) (end 154.85 112.6) (width 0.1524) (layer F.Cu) (net 1))
-  (segment (start 155.025 113.5) (end 154.85 113.325) (width 0.1524) (layer F.Cu) (net 1))
   (segment (start 155.15 113.55) (end 155.2 113.5) (width 0.1524) (layer F.Cu) (net 1))
   (segment (start 155.5 112.3) (end 155.5 113.4) (width 0.1524) (layer F.Cu) (net 1))
@@
   (segment (start 186.084238 102.8) (end 186.3 102.8) (width 0.1524) (layer B.Cu) (net 1))
   (segment (start 186.3 102.8) (end 187.45 101.65) (width 0.1524) (layer B.Cu) (net 1))
-  (segment (start 159.2 109.9) (end 158 111.1) (width 0.1524) (layer B.Cu) (net 1))
-  (segment (start 158 111.1) (end 158 111.96) (width 0.1524) (layer B.Cu) (net 1))
-  (segment (start 159.75882 109.9) (end 159.2 109.9) (width 0.1524) (layer B.Cu) (net 1))
-  (segment (start 159.77941 109.92059) (end 159.75882 109.9) (width 0.1524) (layer B.Cu) (net 1))
-  (segment (start 168.32941 109.92059) (end 159.77941 109.92059) (width 0.1524) (layer B.Cu) (net 1))
   (segment (start 169.35 108.8) (end 169.35 108.9) (width 0.1524) (layer B.Cu) (net 1))
-  (segment (start 169.35 108.9) (end 168.32941 109.92059) (width 0.1524) (layer B.Cu) (net 1))
   (segment (start 181.45 95.1) (end 180.8976 95.1) (width 0.1524) (layer B.Cu) (net 1))
   (segment (start 180.8976 95.1) (end 179.459806 96.537794) (width 0.1524) (layer B.Cu) (net 1))
@@
   (segment (start 176.403201 100.478537) (end 176.08 100.801738) (width 0.1524) (layer B.Cu) (net 1))
   (segment (start 176.08 100.801738) (end 176.08 101.31) (width 0.1524) (layer B.Cu) (net 1))
-  (segment (start 154.65 112.4) (end 153.55 112.4) (width 0.1524) (layer F.Cu) (net 1))
   (segment (start 178.58 101.31) (end 178.58 102.052997) (width 0.1524) (layer B.Cu) (net 1))
   (segment (start 178.58 102.052997) (end 178.827003 102.3) (width 0.1524) (layer B.Cu) (net 1))
@@
   (segment (start 133.05625 98.797698) (end 131.69375 98.797698) (width 0.1524) (layer B.Cu) (net 1))
   (segment (start 131.69375 98.797698) (end 131.5875 98.903948) (width 0.1524) (layer B.Cu) (net 1))
-  (segment (start 124.8976 108.7) (end 131.4 108.7) (width 0.1524) (layer B.Cu) (net 1))
-  (segment (start 131.4 108.7) (end 132.1 108) (width 0.1524) (layer B.Cu) (net 1))
-  (segment (start 132.1 108) (end 132.1 107.95) (width 0.1524) (layer B.Cu) (net 1))
-  (segment (start 124.6 107.95) (end 124.6 108.4024) (width 0.1524) (layer B.Cu) (net 1))
-  (segment (start 124.6 108.4024) (end 124.8976 108.7) (width 0.1524) (layer B.Cu) (net 1))
   (segment (start 129.4 97.25) (end 131.403948 97.25) (width 0.508) (layer F.Cu) (net 1))
   (segment (start 131.403948 97.25) (end 131.90625 96.747698) (width 0.508) (layer F.Cu) (net 1))
@@
   (segment (start 145.95 120.35) (end 145.130001 119.530001) (width 0.508) (layer F.Cu) (net 16))
   (segment (start 145.130001 119.530001) (end 145.100001 119.530001) (width 0.508) (layer F.Cu) (net 16))
+  (segment (start 145.95 117.84) (end 146.8 116.99) (width 0.508) (layer F.Cu) (net 17))
+  (segment (start 146.8 116.99) (end 147.651769 116.138231) (width 0.1524) (layer F.Cu) (net 17))
   (segment (start 161.1 104.98) (end 160.849999 104.729999) (width 0.1524) (layer F.Cu) (net 17))
   (segment (start 161.1 108.2) (end 161.1 104.98) (width 0.1524) (layer F.Cu) (net 17))
@@
   (segment (start 158.138233 114.647205) (end 158.138233 111.161767) (width 0.1524) (layer F.Cu) (net 17))
   (segment (start 147.651769 116.138231) (end 156.647207 116.138231) (width 0.1524) (layer F.Cu) (net 17))
-  (segment (start 145.95 117.84) (end 147.651769 116.138231) (width 0.1524) (layer F.Cu) (net 17))
   (segment (start 160.849999 104.729999) (end 160.6 104.48) (width 0.1524) (layer F.Cu) (net 17))
   (segment (start 156.647207 116.138231) (end 158.138233 114.647205) (width 0.1524) (layer F.Cu) (net 17))
